Commit message: Update joint limits and link properties in URDF
Actualización de datos de inercia del gripper

File: urdf/dofbotpi5.urdf (robot description, URDF)
Before this commit: robot dofbotpi5, 9 links, 8 joints
Links:
- link link_5: mass 0.03523 -> 0.04738955
Joints:
- joint j1: limit lower=-3.1415 upper=3.1415 effort=10.0 velocity=2.0 -> lower=-1.5708 upper=1.5708 effort=10.0 velocity=2.0
- joint j2: limit lower=-3.1415 upper=3.1415 effort=10.0 velocity=2.0 -> lower=-1.5708 upper=1.5708 effort=10.0 velocity=2.0
- joint j3: limit lower=-3.1415 upper=3.1415 effort=10.0 velocity=2.0 -> lower=-2.3911 upper=1.7453 effort=10.0 velocity=2.0
- joint j4: limit lower=-3.1415 upper=3.1415 effort=10.0 velocity=2.0 -> lower=-1.5708 upper=1.5708 effort=10.0 velocity=2.0
- joint j45: limit lower=-3.1415 upper=3.1415 effort=10.0 velocity=2.0 -> lower=-1.5708 upper=3.1416 effort=10.0 velocity=2.0
